File: Proiect Paul/memorii/test.sch (KiCad schematic (older format))
At the start: 10 parts

Commit message: Good things
Parts:
- Decodificator: symbol PMD:74AC11138 -> test-rescue:74AC11138-PMD
- SRAM0, SRAM1, SRAM2, SRAM3: symbol PMD:62256 -> test-rescue:62256-PMD
Changed lines of the file:
@@
 $EndComp
 $Comp
-L PMD:62256 SRAM1
+L test-rescue:62256-PMD SRAM1
 U 1 1 5BF9B82B
 P 8991 4465
@@
 $EndComp
 $Comp
-L PMD:62256 SRAM2
+L test-rescue:62256-PMD SRAM2
 U 1 1 5BF9B884
 P 10543 4465
@@
 $EndComp
 $Comp
-L PMD:62256 SRAM3
+L test-rescue:62256-PMD SRAM3
 U 1 1 5BF9B92A
 P 12082 4454
@@
 RD
 $Comp
-L PMD:74AC11138 Decodificator
+L test-rescue:74AC11138-PMD Decodificator
 U 1 1 5DE813C1
 P 1499 5718
@@
 Connection ~ 6028 3816
 $Comp
-L PMD:62256 SRAM0
+L test-rescue:62256-PMD SRAM0
 U 1 1 5BF9B730
 P 7528 4466
