File: Proiect Paul/pmd3_procesor/pmd3_procesor.sch (KiCad schematic (older format))
At the start: 11 parts

Commit message: Good things
Parts:
- U?: symbol MCU_Intel:8086_Max_Mode -> pmd3_procesor-rescue:8086_Max_Mode-MCU_Intel
- U? (x3): symbol 74xx:74LS373 -> pmd3_procesor-rescue:74LS373-74xx
- U? (x2): symbol 74xx:74LS245 -> pmd3_procesor-rescue:74LS245-74xx
Changed lines of the file:
@@
 $EndComp
 $Comp
-L 74xx:74LS373 U?
+L pmd3_procesor-rescue:74LS373-74xx U?
 U 1 1 5C245DB6
 P 16000 2500
@@
 $EndComp
 $Comp
-L 74xx:74LS373 U?
+L pmd3_procesor-rescue:74LS373-74xx U?
 U 1 1 5C245E28
 P 16050 5900
@@
 $EndComp
 $Comp
-L 74xx:74LS373 U?
+L pmd3_procesor-rescue:74LS373-74xx U?
 U 1 1 5C245E85
 P 16000 7550
@@
 $EndComp
 $Comp
-L 74xx:74LS245 U?
+L pmd3_procesor-rescue:74LS245-74xx U?
 U 1 1 5C245F0B
 P 16050 9700
@@
 $EndComp
 $Comp
-L 74xx:74LS245 U?
+L pmd3_procesor-rescue:74LS245-74xx U?
 U 1 1 5C245F86
 P 16050 11900
@@
 RST
 $Comp
-L MCU_Intel:8086_Max_Mode U?
+L pmd3_procesor-rescue:8086_Max_Mode-MCU_Intel U?
 U 1 1 5C1E9592
 P 7550 5200
