File: Proiect Paul/pmd_afisaje/pmd.sch (KiCad schematic (older format))
At the start: 113 parts

Commit message: Good things
Parts:
- U? (x2): symbol PMD:5OR -> pmd-rescue:5OR-PMD
- U? (x2): symbol PMD:6NOR -> pmd-rescue:6NOR-PMD
Changed lines of the file:
@@
 	1280 10047 636  10047
 $Comp
-L PMD:5OR U?
+L pmd-rescue:5OR-PMD U?
 U 1 1 5DE3AD6A
 P 1476 5692
@@
 A6
 $Comp
-L PMD:6NOR U?
+L pmd-rescue:6NOR-PMD U?
 U 1 1 5DF9DAE4
 P 1458 6347
@@
 	1038 6172 1134 6172
 $Comp
-L PMD:5OR U?
+L pmd-rescue:5OR-PMD U?
 U 1 1 5E2378F2
 P 1692 13147
@@
 A6
 $Comp
-L PMD:6NOR U?
+L pmd-rescue:6NOR-PMD U?
 U 1 1 5E2D68E6
 P 2347 13919
