File: diana/afis/afis.sch (KiCad schematic (older format))
At the start: 76 parts

Commit message: Afis
Parts:
- removed D? (x16): D, symbol Device:D
- removed D? (x4): BAY93, Diode_THT:D_DO-35_SOD27_P7.62mm_Horizontal, symbol Diode:BAY93
- removed R? (x20): R, symbol Device:R
- removed SW? (x16): SW_Push, symbol Switch:SW_Push
- removed U? (x8): KCSC02-105, Display_7Segment:KCSC02-105, symbol Display_Character:KCSC02-105
- removed U? (x11): 74HCT574, symbol 74xx:74HCT574
- removed U?: 74x244, symbol afis_lib:74x244
- added D? (x8): HD7731, HD7731, symbol pmd-rescue:HD7731-Display_Character
- added D? (x18): D, symbol Device:D
- added Rez_8x? (x26): R_Small, symbol Device:R_Small
- added SW? (x16): SW_Push, symbol Switch:SW_Push
- added U? (x11): 74LS373, symbol pmd-rescue:74LS373-74xx
- added U?: 5OR, symbol pmd-rescue:5OR-PMD
- added U?: 74LS244N, symbol pmd-rescue:74LS244N-74xx
- added U?: 6NOR, symbol pmd-rescue:6NOR-PMD
- added U?: 74LS32, symbol 74xx:74LS32
- added U?: 74159, symbol pmd-rescue:74159-74xx_IEEE
Connections:
- net labels added: "1", 4x10k, A0, A1, A10, A11, A12, A13, A14, A15, A2, A3, A4, A5, A6, A7, A8, A9, M\~IO, Vcc
- net labels removed: VCC
- wire segments 356 -> 359
- no-connect marks 1 -> 0
Other:
- note removed: "D7-D0"
- note removed: "Magistrala de date"

Commit message: chestii
Parts:
- added D? (x2): D, symbol Device:D
- added Rez_8x? (x2): R_Small, symbol Device:R_Small
- D? (x8): symbol pmd-rescue:HD7731-Display_Character -> afis-rescue:HD7731-Display_Character-pmd-rescue
- U? (x11): symbol pmd-rescue:74LS373-74xx -> afis-rescue:74LS373-74xx-pmd-rescue
- U?: symbol pmd-rescue:5OR-PMD -> afis-rescue:5OR-PMD-pmd-rescue
- U?: symbol pmd-rescue:74LS244N-74xx -> afis-rescue:74LS244N-74xx-pmd-rescue
- U?: symbol pmd-rescue:6NOR-PMD -> afis-rescue:6NOR-PMD-pmd-rescue
- U?: symbol pmd-rescue:74159-74xx_IEEE -> afis-rescue:74159-74xx_IEEE-pmd-rescue
Connections:
- wire segments 359 -> 358
Changed lines of the file:
@@
 EESchema Schematic File Version 4
 LIBS:afis-cache
-LIBS:pmd-cache
 EELAYER 26 0
 EELAYER END
@@
 $EndDescr
 $Comp
-L pmd-rescue:HD7731-Display_Character D?
+L afis-rescue:HD7731-Display_Character-pmd-rescue D?
 U 1 1 5C10F59D
 P 11384 6160
@@
 $EndComp
 $Comp
-L pmd-rescue:HD7731-Display_Character D?
+L afis-rescue:HD7731-Display_Character-pmd-rescue D?
 U 1 1 5C10F5A4
 P 13934 6160
@@
 $EndComp
 $Comp
-L pmd-rescue:HD7731-Display_Character D?
+L afis-rescue:HD7731-Display_Character-pmd-rescue D?
 U 1 1 5C10F5AB
 P 16634 6160
@@
 $EndComp
 $Comp
-L pmd-rescue:HD7731-Display_Character D?
+L afis-rescue:HD7731-Display_Character-pmd-rescue D?
 U 1 1 5C10F5B2
 P 19234 6160
@@
 $EndComp
 $Comp
-L pmd-rescue:HD7731-Display_Character D?
+L afis-rescue:HD7731-Display_Character-pmd-rescue D?
 U 1 1 5C10F5B9
 P 21684 6160
@@
 $EndComp
 $Comp
-L pmd-rescue:HD7731-Display_Character D?
+L afis-rescue:HD7731-Display_Character-pmd-rescue D?
 U 1 1 5C10F5C0
 P 24034 6160
@@
 $EndComp
 $Comp
-L pmd-rescue:HD7731-Display_Character D?
+L afis-rescue:HD7731-Display_Character-pmd-rescue D?
 U 1 1 5C10F5C7
 P 26334 6160
@@
 $EndComp
 $Comp
-L pmd-rescue:HD7731-Display_Character D?
+L afis-rescue:HD7731-Display_Character-pmd-rescue D?
 U 1 1 5C10F5CE
 P 28784 6160
@@
 $EndComp
 $Comp
-L pmd-rescue:74LS373-74xx U?
+L afis-rescue:74LS373-74xx-pmd-rescue U?
 U 1 1 5C10F5DC
 P 13584 7460
@@
 $EndComp
 $Comp
-L pmd-rescue:74LS373-74xx U?
+L afis-rescue:74LS373-74xx-pmd-rescue U?
 U 1 1 5C10F5E3
 P 16434 7460
@@
 $EndComp
 $Comp
-L pmd-rescue:74LS373-74xx U?
+L afis-rescue:74LS373-74xx-pmd-rescue U?
 U 1 1 5C10F5EA
 P 18984 7510
@@
 $EndComp
 $Comp
-L pmd-rescue:74LS373-74xx U?
+L afis-rescue:74LS373-74xx-pmd-rescue U?
 U 1 1 5C10F5F1
 P 21434 7610
@@
 $EndComp
 $Comp
-L pmd-rescue:74LS373-74xx U?
+L afis-rescue:74LS373-74xx-pmd-rescue U?
 U 1 1 5C10F5F8
 P 23634 7610
@@
 $EndComp
 $Comp
-L pmd-rescue:74LS373-74xx U?
+L afis-rescue:74LS373-74xx-pmd-rescue U?
 U 1 1 5C10F5FF
 P 26184 7660
@@
 $EndComp
 $Comp
-L pmd-rescue:74LS373-74xx U?
+L afis-rescue:74LS373-74xx-pmd-rescue U?
 U 1 1 5C10F606
 P 28384 7660
@@
 Wire Wire Line
 	12534 5810 12534 4960
-Connection ~ 9984 4360
 Connection ~ 9984 4810
 Wire Wire Line
@@
 Connection ~ 27384 4360
 $Comp
-L pmd-rescue:74LS373-74xx U?
+L afis-rescue:74LS373-74xx-pmd-rescue U?
 U 1 1 5C1D1100
 P 30634 6260
@@
 $EndComp
 $Comp
-L pmd-rescue:74LS373-74xx U?
+L afis-rescue:74LS373-74xx-pmd-rescue U?
 U 1 1 5C29341E
 P 30634 9810
@@
 $EndComp
 $Comp
-L pmd-rescue:74LS373-74xx U?
+L afis-rescue:74LS373-74xx-pmd-rescue U?
 U 1 1 5C2C3D60
 P 9206 11236
@@
 Wire Bus Line
 	10384 9010 8984 9010
-Wire Wire Line
-	9684 4360 9984 4360
-$Comp
-L pmd-rescue:74LS244N-74xx U?
+$Comp
+L afis-rescue:74LS244N-74xx-pmd-rescue U?
 U 1 1 5DF5E0B4
 P 28106 11036
@@
 	8706 10186 8706 11436
 $Comp
-L pmd-rescue:74159-74xx_IEEE U?
+L afis-rescue:74159-74xx_IEEE-pmd-rescue U?
 U 1 1 5FC4A75D
 P 3594 7126
@@
 Connection ~ 11534 7060
 $Comp
-L pmd-rescue:74LS373-74xx U?
+L afis-rescue:74LS373-74xx-pmd-rescue U?
 U 1 1 5C10F5D5
 P 11034 7560
@@
 M\~IO
 $Comp
-L pmd-rescue:5OR-PMD U?
+L afis-rescue:5OR-PMD-pmd-rescue U?
 U 1 1 5DE3AD6A
 P 1860 5302
@@
 A6
 $Comp
-L pmd-rescue:6NOR-PMD U?
+L afis-rescue:6NOR-PMD-pmd-rescue U?
 U 1 1 5DF9DAE4
 P 1842 5957
@@
 Wire Wire Line
 	1022 7527 3046 7527
+$Comp
+L Device:R_Small Rez_8x?
+U 1 1 5C0F977B
+P 31534 10010
+F 0 "Rez_8x?" V 31638 10010 50  0001 C CNN
+F 1 "R_Small" V 31639 10010 50  0001 C CNN
+F 2 "" H 31534 10010 50  0001 C CNN
+F 3 "~" H 31534 10010 50  0001 C CNN
+	1    31534 10010
+	0    -1   -1   0
+$EndComp
+$Comp
+L Device:R_Small Rez_8x?
+U 1 1 5C0F9781
+P 31534 9910
+F 0 "Rez_8x?" V 31638 9910 50  0001 C CNN
+F 1 "R_Small" V 31639 9910 50  0001 C CNN
+F 2 "" H 31534 9910 50  0001 C CNN
+F 3 "~" H 31534 9910 50  0001 C CNN
+	1    31534 9910
+	0    -1   -1   0
+$EndComp
+$Comp
+L Device:D D?
+U 1 1 5C0F9787
+P 31284 9910
+F 0 "D?" H 31284 10034 50  0001 C CNN
+F 1 "D" H 31284 10035 50  0001 C CNN
+F 2 "" H 31284 9910 50  0001 C CNN
+F 3 "~" H 31284 9910 50  0001 C CNN
+	1    31284 9910
+	1    0    0    -1
+$EndComp
+$Comp
+L Device:D D?
+U 1 1 5C0F978D
+P 31284 10010
+F 0 "D?" H 31284 10134 50  0001 C CNN
+F 1 "D" H 31284 10135 50  0001 C CNN
+F 2 "" H 31284 10010 50  0001 C CNN
+F 3 "~" H 31284 10010 50  0001 C CNN
+	1    31284 10010
+	1    0    0    -1
+$EndComp
 $EndSCHEMATC

Commit message: c
Parts:
- removed U?: 6NOR, symbol afis-rescue:6NOR-PMD-pmd-rescue
- added U? (x4): 74LS32, symbol 74xx:74LS32
- added U? (x3): 74LS04, symbol 74xx:74LS04
Connections:
- net labels removed: "1"
- wire segments 358 -> 373
Other:
- moved on the sheet: U?, U?A
Changed lines of the file:
@@
 L afis-rescue:5OR-PMD-pmd-rescue U?
 U 1 1 5DE3AD6A
-P 1860 5302
-F 0 "U?" H 1835 5877 50  0000 C CNN
-F 1 "5OR" H 1835 5786 50  0000 C CNN
-F 2 "" H 1810 5352 50  0001 C CNN
-F 3 "" H 1810 5352 50  0001 C CNN
-	1    1860 5302
-	1    0    0    -1
-$EndComp
-Text Label 1442 4962 0    39   ~ 0
+P 1202 4688
+F 0 "U?" H 1177 5263 50  0000 C CNN
+F 1 "5OR" H 1177 5172 50  0000 C CNN
+F 2 "" H 1152 4738 50  0001 C CNN
+F 3 "" H 1152 4738 50  0001 C CNN
+	1    1202 4688
+	0    1    1    0
+$EndComp
+Text Label 1542 4270 3    39   ~ 0
 A15
-Text Label 1431 5023 0    39   ~ 0
+Text Label 1481 4259 3    39   ~ 0
 A14
-Text Label 1430 5073 0    39   ~ 0
+Text Label 1431 4258 3    39   ~ 0
 A13
-Text Label 1433 5124 0    39   ~ 0
+Text Label 1380 4261 3    39   ~ 0
 A12
-Text Label 1438 5178 0    39   ~ 0
+Text Label 1326 4266 3    39   ~ 0
 A10
-Text Label 1421 5233 0    39   ~ 0
-A5
-Text Label 1436 4910 0    39   ~ 0
-A4
-Text Label 1392 5510 0    39   ~ 0
-A11
-Text Label 1470 5570 0    39   ~ 0
+Text Label 1271 4249 3    39   ~ 0
 A9
-Text Label 1473 5621 0    39   ~ 0
+Text Label 1594 4264 3    39   ~ 0
 A8
-Text Label 1479 5667 0    39   ~ 0
-A7
-Text Label 1479 5714 0    39   ~ 0
-A6
-$Comp
-L afis-rescue:6NOR-PMD-pmd-rescue U?
-U 1 1 5DF9DAE4
-P 1842 5957
-F 0 "U?" H 1842 6633 39  0000 C CNN
-F 1 "6NOR" H 1842 6558 39  0000 C CNN
-F 2 "" H 1842 5957 39  0001 C CNN
-F 3 "" H 1842 5957 39  0001 C CNN
-	1    1842 5957
-	1    0    0    -1
-$EndComp
 $Comp
 L 74xx:74LS32 U?
 U 1 1 5E02C74C
-P 2680 5328
-F 0 "U?" H 2680 5653 50  0000 C CNN
-F 1 "74LS32" H 2680 5562 50  0000 C CNN
-F 2 "" H 2680 5328 50  0001 C CNN
-F 3 "http://www.ti.com/lit/gpn/sn74LS32" H 2680 5328 50  0001 C CNN
-	1    2680 5328
-	1    0    0    -1
-$EndComp
-Wire Wire Line
-	2160 5052 2269 5052
-Wire Wire Line
-	2269 5052 2269 5228
-Wire Wire Line
-	2269 5228 2380 5228
-Connection ~ 2380 5228
-Wire Wire Line
-	2380 5228 2382 5228
-Wire Wire Line
-	2381 5428 2380 5428
-Wire Wire Line
-	2219 5428 2219 5632
-Wire Wire Line
-	2219 5632 2166 5632
-Connection ~ 2380 5428
-Wire Wire Line
-	2380 5428 2219 5428
-Wire Wire Line
-	2980 5328 3046 5328
-Wire Wire Line
-	3046 5328 3046 5594
-Wire Wire Line
-	3046 5594 2751 5594
-Wire Wire Line
-	2751 5594 2751 7726
-Wire Wire Line
-	2751 7726 3044 7726
+P 1176 5508
+F 0 "U?" H 1176 5833 50  0000 C CNN
+F 1 "74LS32" H 1176 5742 50  0000 C CNN
+F 2 "" H 1176 5508 50  0001 C CNN
+F 3 "http://www.ti.com/lit/gpn/sn74LS32" H 1176 5508 50  0001 C CNN
+	1    1176 5508
+	0    1    1    0
+$EndComp
+Wire Wire Line
+	1452 4988 1452 5097
+Wire Wire Line
+	1452 5097 1276 5097
+Wire Wire Line
+	1276 5097 1276 5208
+Connection ~ 1276 5208
+Wire Wire Line
+	1276 5208 1276 5210
+Wire Wire Line
+	1076 5209 1076 5208
+Wire Wire Line
+	1076 5047 872  5047
+Wire Wire Line
+	872  5047 872  4995
+Connection ~ 1076 5208
+Wire Wire Line
+	1076 5208 1076 5047
 Connection ~ 3044 7726
 Wire Wire Line
 	3044 7726 3047 7726
-Text GLabel 1363 5720 0    50   Input ~ 0
-"1"
-Wire Wire Line
-	1364 5720 1410 5720
-Wire Wire Line
-	1410 5720 1410 5732
-Wire Wire Line
-	1410 5732 1569 5732
-Wire Wire Line
-	1422 5731 1422 5782
-Wire Wire Line
-	1422 5782 1518 5782
 Wire Wire Line
 	10014 8061 10538 8061
@@
 Wire Wire Line
 	8706 11736 8710 11736
-Wire Wire Line
-	4142 7425 8478 7425
 Wire Wire Line
 	8478 7425 8478 12120
@@
 	1    0    0    -1
 $EndComp
+$Comp
+L 74xx:74LS32 U?
+U 1 1 5C8F4EE7
+P 2044 4690
+F 0 "U?" H 2044 5015 50  0000 C CNN
+F 1 "74LS32" H 2044 4924 50  0000 C CNN
+F 2 "" H 2044 4690 50  0001 C CNN
+F 3 "http://www.ti.com/lit/gpn/sn74LS32" H 2044 4690 50  0001 C CNN
+	1    2044 4690
+	0    1    1    0
+$EndComp
+Text Label 1914 4282 3    39   ~ 0
+A11
+Text Label 2120 4304 3    39   ~ 0
+A5
+$Comp
+L 74xx:74LS32 U?
+U 1 1 5C942EF5
+P 1944 5290
+F 0 "U?" H 1944 5615 50  0000 C CNN
+F 1 "74LS32" H 1944 5524 50  0000 C CNN
+F 2 "" H 1944 5290 50  0001 C CNN
+F 3 "http://www.ti.com/lit/gpn/sn74LS32" H 1944 5290 50  0001 C CNN
+	1    1944 5290
+	0    1    1    0
+$EndComp
+Text Label 1825 4823 3    39   ~ 0
+A4
+$Comp
+L 74xx:74LS32 U?
+U 1 1 5C9B81C8
+P 1641 6417
+F 0 "U?" V 1595 6605 50  0000 L CNN
+F 1 "74LS32" V 1686 6605 50  0000 L CNN
+F 2 "" H 1641 6417 50  0001 C CNN
+F 3 "http://www.ti.com/lit/gpn/sn74LS32" H 1641 6417 50  0001 C CNN
+	1    1641 6417
+	0    1    1    0
+$EndComp
+Wire Wire Line
+	1175 5808 1176 5808
+Wire Wire Line
+	1541 5808 1541 6117
+Connection ~ 1176 5808
+Wire Wire Line
+	1176 5808 1541 5808
+Wire Wire Line
+	1741 6118 1741 6117
+Wire Wire Line
+	1741 5815 1943 5815
+Wire Wire Line
+	1943 5815 1943 5590
+Connection ~ 1741 6117
+Wire Wire Line
+	1741 6117 1741 5815
+$Comp
+L 74xx:74LS32 U?
+U 1 1 5CE479B7
+P 872 4695
+F 0 "U?" V 826 4883 50  0000 L CNN
+F 1 "74LS32" V 917 4883 50  0000 L CNN
+F 2 "" H 872 4695 50  0001 C CNN
+F 3 "http://www.ti.com/lit/gpn/sn74LS32" H 872 4695 50  0001 C CNN
+	1    872  4695
+	0    1    1    0
+$EndComp
+Connection ~ 872  4995
+Wire Wire Line
+	872  4995 872  4994
+Text Label 798  3530 1    50   ~ 0
+A7
+Text Label 1131 3550 1    50   ~ 0
+A6
+$Comp
+L 74xx:74LS04 U?
+U 1 1 5CE96FE8
+P 754 3867
+F 0 "U?" V 708 4047 50  0000 L CNN
+F 1 "74LS04" V 799 4047 50  0000 L CNN
+F 2 "" H 754 3867 50  0001 C CNN
+F 3 "http://www.ti.com/lit/gpn/sn74LS04" H 754 3867 50  0001 C CNN
+	1    754  3867
+	0    1    1    0
+$EndComp
+$Comp
+L 74xx:74LS04 U?
+U 1 1 5CE97134
+P 1096 3873
+F 0 "U?" V 1050 4053 50  0000 L CNN
+F 1 "74LS04" V 1141 4053 50  0000 L CNN
+F 2 "" H 1096 3873 50  0001 C CNN
+F 3 "http://www.ti.com/lit/gpn/sn74LS04" H 1096 3873 50  0001 C CNN
+	1    1096 3873
+	0    1    1    0
+$EndComp
+Wire Wire Line
+	753  4164 753  4361
+Wire Wire Line
+	753  4361 772  4361
+Wire Wire Line
+	772  4361 772  4395
+Connection ~ 772  4395
+Wire Wire Line
+	772  4395 772  4397
+Wire Wire Line
+	1096 4171 1096 4173
+Wire Wire Line
+	1096 4333 972  4333
+Wire Wire Line
+	972  4333 972  4395
+Connection ~ 1096 4173
+Wire Wire Line
+	1096 4173 1096 4333
+Connection ~ 972  4395
+Wire Wire Line
+	972  4395 972  4396
+Wire Wire Line
+	1640 6714 1640 7726
+Wire Wire Line
+	1640 7726 3044 7726
+$Comp
+L 74xx:74LS04 U?
+U 1 1 5CF9A114
+P 6012 7576
+F 0 "U?" H 6012 7893 50  0000 C CNN
+F 1 "74LS04" H 6012 7802 50  0000 C CNN
+F 2 "" H 6012 7576 50  0001 C CNN
+F 3 "http://www.ti.com/lit/gpn/sn74LS04" H 6012 7576 50  0001 C CNN
+	1    6012 7576
+	1    0    0    -1
+$EndComp
+Wire Wire Line
+	4142 7427 5478 7427
+Wire Wire Line
+	5478 7427 5478 7580
+Wire Wire Line
+	5478 7580 5712 7580
+Wire Wire Line
+	6310 7576 6312 7576
+Wire Wire Line
+	6392 7576 6392 7424
+Wire Wire Line
+	6392 7424 8478 7424
+Connection ~ 6312 7576
+Wire Wire Line
+	6312 7576 6392 7576
 $EndSCHEMATC
